Commit message: Created DRIVE ROBOT SIMU

File: description/robot_core.xacro (robot description, xacro)
@@ -27,5 +27,5 @@
             <origin xyz="0.115 0 0.025"/> <!-- ubicacion dentro de la caja-->
                 <geometry>
-                    <box size="0.23 0.19 0.01"/>
+                    <box size="0.23 0.19 0.02"/>
                 </geometry>
                 <material name="white"/>
@@ -41,9 +41,12 @@
         </xacro:inertial_box>
     </link>
+    <gazebo reference="chassis">
+        <material>Gazebo/White</material>
+    </gazebo>
     <!-- LEFT WHEEL LINK -->
     <joint name="left_wheel_joint" type="continuous">
         <parent link="base_link"/>
         <child link="left_wheel"/>
-        <origin xyz="0 -0.1 0" rpy="${pi/2} 0 0"/>
+        <origin xyz="0 -0.11 0" rpy="${pi/2} 0 0"/>
         <axis xyz="0 0 1"/>
     </joint>
@@ -64,9 +67,12 @@
         </xacro:inertial_cylinder>
     </link>
+    <gazebo reference="left_wheel">
+        <material>Gazebo/Blue</material>
+    </gazebo>
    <!-- RIGHT WHEEL LINK -->
    <joint name="right_wheel_joint" type="continuous">
         <parent link="base_link"/>
         <child link="right_wheel"/>
-        <origin xyz="0 0.1 0" rpy="-${pi/2} 0 0"/>
+        <origin xyz="0 0.11 0" rpy="-${pi/2} 0 0"/>
         <axis xyz="0 0 -1"/>
     </joint>
@@ -87,4 +93,7 @@
         </xacro:inertial_cylinder>
     </link>
+    <gazebo reference="right_wheel">
+        <material>Gazebo/Blue</material>
+    </gazebo>
   <!-- CASTER WHEEL LINK -->
     <joint name="caster_wheel_joint" type="fixed">
@@ -109,3 +118,8 @@
         </xacro:inertial_sphere>
     </link>
+    <gazebo reference="caster_wheel">
+        <material>Gazebo/Black</material>
+        <mu1 value="0.001"/>
+        <mu2 value="0.001"/>
+    </gazebo>
 </robot>
