Commit message: Extra bits

File: description/robot.urdf.xacro (robot description, xacro)
@@ -1,6 +1,12 @@
 <?xml version="1.0"?>
 <robot xmlns:xacro="http://www.ros.org/wiki/xacro"  name="robot">
+    <xacro:arg name="use_ros2_control" default="true"/>
+    <xacro:arg name="sim_mode" default="false"/>
     <xacro:include filename="robot_core.xacro" />
-    <!-- <xacro:include filename="gazebo_control.xacro" /> -->
-    <xacro:include filename="ros2_control.xacro" />
+    <xacro:if value="$(arg use_ros2_control)">
+        <xacro:include filename="ros2_control.xacro" />
+    </xacro:if>
+    <xacro:unless value="$(arg use_ros2_control)">
+        <xacro:include filename="gazebo_control.xacro" />
+    </xacro:unless>
 </robot>

File: description/robot_core.xacro (robot description, xacro)
@@ -2,45 +2,62 @@
 <robot xmlns:xacro="http://www.ros.org/wiki/xacro" >
     <xacro:include filename="inertial_macros.xacro"/>
+    <xacro:property name="chassis_length" value="0.23"/>
+    <xacro:property name="chassis_width" value="0.19"/>
+    <xacro:property name="chassis_height" value="0.02"/>
+    <xacro:property name="chassis_mass" value="1.335"/>
+    <xacro:property name="wheel_radius" value="0.03325"/>
+    <xacro:property name="wheel_thickness" value="0.0266"/>
+    <xacro:property name="wheel_mass" value="0.03"/>
+    <xacro:property name="wheel_offset_x" value="0.02"/>
+    <xacro:property name="wheel_offset_y" value="0.11"/>
+    <xacro:property name="wheel_offset_z" value="0"/>
+    <xacro:property name="caster_wheel_radius" value="0.02"/>
+    <xacro:property name="caster_wheel_mass" value="0.03"/>
+    <xacro:property name="caster_wheel_offset_x" value="0.19"/>
+    <!--<xacro:property name="caster_wheel_offset_z" value="${wheel_offset_z - wheel_radius + caster_wheel_radius}"/> -->
     <material name="white">
         <color rgba="1 1 1 1" />
     </material>
     <material name="orange">
-        <color rgba="1 0.3 0.1 1" />
+        <color rgba="1 0.3 0.1 1"/>
     </material>
     <material name="blue">
-        <color rgba="0.2 0.2 1 1" />
+        <color rgba="0.2 0.2 1 1"/>
     </material>
     <material name="black">
-        <color rgba="0 0 0 1" />
+        <color rgba="0 0 0 1"/>
     </material>
-    <!-- base link -->
+    <material name="red">
+        <color rgba="1 0 0 1"/>
+    </material>
+    <!-- BASE LINK -->
     <link name="base_link">
     </link>
-    <!-- chasis link -->
+    <!-- CHASSIS LINK -->
     <joint name="chassis_joint" type="fixed">
         <parent link="base_link"/>
         <child link="chassis"/>
-        <origin xyz="-0.02 0 0"/><!-- desfase de eje de rueda y origen-->
+        <origin xyz="-${wheel_offset_x} 0 ${-wheel_offset_z}"/>
     </joint>
     <link name="chassis">
         <visual>
-            <origin xyz="0.115 0 0.025"/> <!-- ubicacion dentro de la caja-->
-                <geometry>
-                    <box size="0.23 0.19 0.02"/>
-                </geometry>
-                <material name="white"/>
+            <origin xyz="${chassis_length/2} 0 0.025"/>
+            <geometry>
+                <box size="${chassis_length} ${chassis_width} ${chassis_height}"/>
+            </geometry>
+            <material name="orange"/>
         </visual>
         <collision>
-            <origin xyz="0.115 0 0.025"/>
-                <geometry>
-                    <box size="0.23 0.19 0.01"/>
-                </geometry>
+            <origin xyz="${chassis_length/2} 0 ${chassis_height/2}"/>
+            <geometry>
+                <box size="${chassis_length} ${chassis_width} ${chassis_height}"/>
+            </geometry>
         </collision>
-        <xacro:inertial_box mass="1.355" x="0.23" y="0.19" z="0.01">
-            <origin xyz="0.115 0 0.025" rpy="0 0 0"/>
+        <xacro:inertial_box mass="0.5" x="${chassis_length}" y="${chassis_width}" z="${chassis_height}">
+            <origin xyz="${chassis_length/2} 0 ${chassis_height/2}" rpy="0 0 0"/>
         </xacro:inertial_box>
     </link>
     <gazebo reference="chassis">
-        <material>Gazebo/White</material>
+        <material>Gazebo/Orange</material>
     </gazebo>
     <!-- LEFT WHEEL LINK -->
@@ -48,20 +65,20 @@
         <parent link="base_link"/>
         <child link="left_wheel"/>
-        <origin xyz="0 -0.11 0" rpy="${pi/2} 0 0"/>
-        <axis xyz="0 0 1"/>
+        <origin xyz="0 ${wheel_offset_y} 0" rpy="-${pi/2} 0 0" />
+        <axis xyz="0 0 -1"/>
     </joint>
     <link name="left_wheel">
         <visual>
             <geometry>
-                <cylinder radius="0.03325" length="0.0266"/>
-            </geometry>       <!-- 0.001 -->
+                <cylinder radius="${wheel_radius}" length="${wheel_thickness}"/>
+            </geometry>
             <material name="blue"/>
         </visual>
         <collision>
             <geometry>
-                <cylinder radius="0.03325" length="0.0266"/>
-            </geometry>       <!-- 0.001 -->
+                <sphere radius="${wheel_radius}"/>
+            </geometry>
         </collision>
-        <xacro:inertial_cylinder mass="0.03" radius="0.03325" length="0.0266">
+        <xacro:inertial_cylinder mass="${wheel_mass}" length="${wheel_thickness}" radius="${wheel_radius}">
             <origin xyz="0 0 0" rpy="0 0 0"/>
         </xacro:inertial_cylinder>
@@ -70,24 +87,24 @@
         <material>Gazebo/Blue</material>
     </gazebo>
-   <!-- RIGHT WHEEL LINK -->
-   <joint name="right_wheel_joint" type="continuous">
+    <!-- RIGHT WHEEL LINK -->
+    <joint name="right_wheel_joint" type="continuous">
         <parent link="base_link"/>
         <child link="right_wheel"/>
-        <origin xyz="0 0.11 0" rpy="-${pi/2} 0 0"/>
-        <axis xyz="0 0 -1"/>
+        <origin xyz="0 ${-wheel_offset_y} 0" rpy="${pi/2} 0 0" />
+        <axis xyz="0 0 1"/>
     </joint>
     <link name="right_wheel">
         <visual>
             <geometry>
-                <cylinder radius="0.03325" length="0.0266"/>
-            </geometry>       <!-- 0.001 -->
+                <cylinder radius="${wheel_radius}" length="${wheel_thickness}"/>
+            </geometry>
             <material name="blue"/>
         </visual>
         <collision>
             <geometry>
-                <cylinder radius="0.03325" length="0.0266"/>
-            </geometry>       <!-- 0.001 -->
+                <sphere radius="${wheel_radius}"/>
+            </geometry>
         </collision>
-        <xacro:inertial_cylinder mass="0.03" radius="0.03325" length="0.0266">
+        <xacro:inertial_cylinder mass="${wheel_mass}" length="${wheel_thickness}" radius="${wheel_radius}">
             <origin xyz="0 0 0" rpy="0 0 0"/>
         </xacro:inertial_cylinder>
@@ -96,28 +113,28 @@
         <material>Gazebo/Blue</material>
     </gazebo>
-  <!-- CASTER WHEEL LINK -->
+    <!-- CASTER WHEEL LINK -->
     <joint name="caster_wheel_joint" type="fixed">
         <parent link="chassis"/>
         <child link="caster_wheel"/>
-        <origin xyz="0.19 0 0"/>
+        <origin xyz="${caster_wheel_offset_x} 0 0"/>
     </joint>
     <link name="caster_wheel">
         <visual>
             <geometry>
-                <sphere radius="0.03325"/>
-            </geometry>       <!-- 0.001 -->
-            <material name="black"/>
+                <sphere radius="${caster_wheel_radius}"/>
+            </geometry>
+            <material name="white"/>
         </visual>
         <collision>
             <geometry>
-                <sphere radius="0.03325"/>
-            </geometry>       <!-- 0.001 -->
+                <sphere radius="${caster_wheel_radius}"/>
+            </geometry>
         </collision>
-        <xacro:inertial_sphere mass="0.03" radius="0.03325">
+        <xacro:inertial_sphere mass="${caster_wheel_mass}" radius="${caster_wheel_radius}">
             <origin xyz="0 0 0" rpy="0 0 0"/>
         </xacro:inertial_sphere>
     </link>
     <gazebo reference="caster_wheel">
-        <material>Gazebo/Black</material>
+        <material>Gazebo/White</material>
         <mu1 value="0.001"/>
         <mu2 value="0.001"/>

File: description/ros2_control.xacro (robot description, xacro)
@@ -25,4 +25,5 @@
         <plugin name="gazebo_ros2_control" filename="libgazebo_ros2_control.so">
             <parameters>$(find my_bot)/config/my_controllers.yaml</parameters>
+            <parameters>$(find my_bot)/config/gaz_ros2_ctl_use_sim.yaml</parameters>
         </plugin>
     </gazebo>
